File: Hardware/Schematic.sch (EAGLE design)
At the start: 102 parts, among them IC1 BD5229G-TR, IC2 XC6220A331MR-G, J1 112A-TAAR-R03_ATTEND, J2 QWIIC_RIGHT_ANGLE, J3 FH34SRJ-24S-0.5SH_99_, J4 SAMACSYS_PARTS_USB4110-GF-A, Q1 20V/4.2A/52mΩ/1.4W, Q2 SI1308EDL-T1-GE3, Q3 20V/4.2A/52mΩ/1.4W, U1 ESP32-C6-WROOM-1-N8, U2 MAX17048G+T10, U3 W25Q512JVEIQ, U4 DS3231SN#

Commit message: fix issues
Parts:
- C25: value 100nF -> 4.7uF
Changed lines of the file:
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@@
 <part name="GND45" library="DeskAssistant v19 v2" library_urn="urn:adsk.wipprod:fs.file:vf.c-uWg7zGRE2SlFihlENo6g" deviceset="GND" device=""/>
 <part name="C24" library="DeskAssistant v19 v2" library_urn="urn:adsk.wipprod:fs.file:vf.c-uWg7zGRE2SlFihlENo6g" deviceset="ESP32_WROVER_EAGLE-LTSPICE_C" device="C0402" value="100nF"/>
-<part name="C25" library="DeskAssistant v19 v2" library_urn="urn:adsk.wipprod:fs.file:vf.c-uWg7zGRE2SlFihlENo6g" deviceset="ESP32_WROVER_EAGLE-LTSPICE_C" device="C0402" value="100nF"/>
+<part name="C25" library="DeskAssistant v19 v2" library_urn="urn:adsk.wipprod:fs.file:vf.c-uWg7zGRE2SlFihlENo6g" deviceset="ESP32_WROVER_EAGLE-LTSPICE_C" device="C0402" value="4.7uF"/>
 <part name="IC2" library="DeskAssistant v19 v2" library_urn="urn:adsk.wipprod:fs.file:vf.c-uWg7zGRE2SlFihlENo6g" deviceset="XC6220A331MR-G" device=""/>
 <part name="C26" library="DeskAssistant v19 v2" library_urn="urn:adsk.wipprod:fs.file:vf.c-uWg7zGRE2SlFihlENo6g" deviceset="ESP32_WROVER_EAGLE-LTSPICE_C" device="C0402" value="4.7uF"/>
@@
 <instance part="D2" gate="G$1" x="-7.62" y="-139.7" smashed="yes" rot="R90">
 <attribute name="NAME" x="-10.16" y="-144.78" size="1.778" layer="95" rot="R90"/>
-<attribute name="VALUE" x="-2.54" y="-144.78" size="1.778" layer="96" rot="R90"/>
+<attribute name="VALUE" x="-2.54" y="-149.86" size="1.778" layer="96" rot="R90"/>
 </instance>
 <instance part="D4" gate="G$1" x="0" y="-139.7" smashed="yes" rot="R90">
-<attribute name="NAME" x="-2.54" y="-144.78" size="1.778" layer="95" rot="R90"/>
-<attribute name="VALUE" x="5.08" y="-144.78" size="1.778" layer="96" rot="R90"/>
+<attribute name="NAME" x="2.54" y="-137.16" size="1.778" layer="95" rot="R90"/>
+<attribute name="VALUE" x="5.08" y="-149.86" size="1.778" layer="96" rot="R90"/>
 </instance>
 <instance part="D6" gate="G$1" x="7.62" y="-139.7" smashed="yes" rot="R90">
-<attribute name="NAME" x="5.08" y="-144.78" size="1.778" layer="95" rot="R90"/>
-<attribute name="VALUE" x="12.7" y="-144.78" size="1.778" layer="96" rot="R90"/>
+<attribute name="NAME" x="10.16" y="-137.16" size="1.778" layer="95" rot="R90"/>
+<attribute name="VALUE" x="12.7" y="-149.86" size="1.778" layer="96" rot="R90"/>
 </instance>
 <instance part="D8" gate="G$1" x="15.24" y="-139.7" smashed="yes" rot="R90">
-<attribute name="NAME" x="12.7" y="-144.78" size="1.778" layer="95" rot="R90"/>
-<attribute name="VALUE" x="20.32" y="-144.78" size="1.778" layer="96" rot="R90"/>
+<attribute name="NAME" x="17.78" y="-137.16" size="1.778" layer="95" rot="R90"/>
+<attribute name="VALUE" x="20.32" y="-149.86" size="1.778" layer="96" rot="R90"/>
 </instance>
 <instance part="D10" gate="G$1" x="22.86" y="-139.7" smashed="yes" rot="R90">
-<attribute name="NAME" x="20.32" y="-144.78" size="1.778" layer="95" rot="R90"/>
-<attribute name="VALUE" x="27.94" y="-144.78" size="1.778" layer="96" rot="R90"/>
+<attribute name="NAME" x="25.4" y="-137.16" size="1.778" layer="95" rot="R90"/>
+<attribute name="VALUE" x="27.94" y="-149.86" size="1.778" layer="96" rot="R90"/>
 </instance>
 <instance part="D11" gate="G$1" x="30.48" y="-139.7" smashed="yes" rot="R90">
-<attribute name="NAME" x="27.94" y="-144.78" size="1.778" layer="95" rot="R90"/>
-<attribute name="VALUE" x="35.56" y="-144.78" size="1.778" layer="96" rot="R90"/>
+<attribute name="NAME" x="33.02" y="-137.16" size="1.778" layer="95" rot="R90"/>
+<attribute name="VALUE" x="35.56" y="-149.86" size="1.778" layer="96" rot="R90"/>
 </instance>
 <instance part="GND18" gate="1" x="-10.16" y="-154.94" smashed="yes">
@@
 <attribute name="NAME" x="21.3614" y="-130.81" size="1.778" layer="95" rot="R90"/>
 <attribute name="NAME" x="21.3614" y="-130.81" size="1.778" layer="95" rot="R90"/>
-<attribute name="VALUE" x="26.162" y="-130.81" size="1.778" layer="96" rot="R90"/>
-<attribute name="VALUE" x="26.162" y="-130.81" size="1.778" layer="96" rot="R90"/>
 </instance>
 <instance part="R6" gate="G$1" x="30.48" y="-127" smashed="yes" rot="R90">
